File: NeepNeep-DAC-V1.kicad_sch (KiCad schematic)
At the start: 18 parts, among them J1 Conn_02x03_Odd_Even, Q1 MMBT3904, U2 W25Q32JVSS, U3 ATtiny85-20SU

Commit message: Commit: M	NeepNeep-DAC-V1.kicad_sch
Other:
- note added: "10k is apparently a good value for this"
- note removed: "This pullup is probably not required but will include anyway"
Changed lines of the file:
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@@
     (effects (font (size 1.27 1.27) (thickness 0.254) bold) (justify left bottom))
   )
-  (text "This pullup is probably\nnot required but will\ninclude anyway"
-    (at 120.65 32.512 0)
+  (text "10k is apparently\na good value \nfor this" (at 120.65 32.512 0)
     (effects (font (size 1.27 1.27)) (justify left bottom))
   )
