File: V2/NeepNeep-DAC-V2.kicad_sch (KiCad schematic)
At the start: 16 parts, among them J1 Conn_02x03_Odd_Even, Q1 MMBT3904, U2 W25Q32JVSS, U3 ATtiny85-20SU

Commit message: Commit: A	V2/NeepNeep-DAC-V2-backups/NeepNeep-DAC-V2-2026-02-09_174934.zip A	V2/NeepNeep-DAC-V2-backups/NeepNeep-DAC-V2-2026-02-10_125359.zip A	V2/NeepNeep-DAC-V2-backups/NeepNeep-DAC-V2-2026-02-10_130055.zip M	V2/NeepNeep-DAC-V2.kicad_pcb M	V2/NeepNeep-DAC-V2.kicad_prl M	V2/NeepNeep-DAC-V2.kicad_sch A	V2/Thumbs.db
Parts:
- removed Q1: MMBT3904, Package_TO_SOT_SMD:SOT-23, symbol Transistor_BJT:MMBT3904
- added Q1: BSS138, Package_TO_SOT_SMD:SOT-23, symbol Transistor_FET:BSS138
- added R4: 100k, Resistor_SMD:R_0805_2012Metric, symbol Device:R
Connections:
- net GND: now also Q1.2 (S), R4.1
- net at BUZZER1.2 (-), C3.2: now also Q1.3 (D)
- net at R7.2: now also Q1.1 (G), R4.2
Other:
- note added: "Added a 100k resistor to ground, apparently this keeps it solidly off when its not being driven."
- note added: "was MMBT3904(RANGE:100-300) (LCSC C20526 or C91032 apparently???) Replace this with a BSS138"
- moved on the sheet: BUZZER1, C3, R7

Commit message: Commit: A	V2/NeepNeep-DAC-V2-backups/NeepNeep-DAC-V2-2026-02-11_154859.zip A	V2/NeepNeep-DAC-V2-backups/NeepNeep-DAC-V2-2026-02-11_164151.zip A	V2/NeepNeep-DAC-V2-backups/NeepNeep-DAC-V2-2026-02-11_165528.zip M	V2/NeepNeep-DAC-V2.kicad_pcb M	V2/NeepNeep-DAC-V2.kicad_prl M	V2/NeepNeep-DAC-V2.kicad_sch
Parts:
- removed JP1: Jumper_2_Open, Connector_PinSocket_1.27mm:PinSocket_1x02_P1.27mm_Vertical, symbol Jumper:Jumper_2_Open
- added J2: Conn_01x03_Pin, Connector_PinHeader_1.27mm:PinHeader_1x03_P1.27mm_Vertical, symbol Connector:Conn_01x03_Pin
Connections:
- net +3V3: now also J2.1 (Pin_1)
- net GND: now also J2.3 (Pin_3)
- net PB3: now also J1.5 (Pin_5)
- net PB5/RESET: now also J2.2 (Pin_2); no longer J1.5 (Pin_5)
Changed lines of the file:
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@@
     )
   )
-  (global_label "PB5{slash}RESET" (shape input) (at 160.02 50.8 180) (fields_autoplaced)
-    (effects (font (size 1.27 1.27)) (justify right))
-    (property "Intersheetrefs" "${INTERSHEET_REFS}" (at 146.8639 50.8 0)
-      (effects (font (size 1.27 1.27)) (justify right) hide)
+  (global_label "PB5{slash}RESET" (shape input) (at 160.782 75.946 0) (fields_autoplaced)
+    (effects (font (size 1.27 1.27)) (justify left))
+    (property "Intersheetrefs" "${INTERSHEET_REFS}" (at 173.9381 75.946 0)
+      (effects (font (size 1.27 1.27)) (justify left) hide)
     )
   )
@@
     (effects (font (size 1.27 1.27)) (justify left))
     (property "Intersheetrefs" "${INTERSHEET_REFS}" (at 105.1337 54.5306 0)
-      (effects (font (size 1.27 1.27)) (justify left) hide)
-    )
-  )
-  (global_label "PB3" (shape input) (at 31.75 135.128 90) (fields_autoplaced)
-    (effects (font (size 1.27 1.27)) (justify left))
-    (property "Intersheetrefs" "${INTERSHEET_REFS}" (at 31.75 129.0475 90)
       (effects (font (size 1.27 1.27)) (justify left) hide)
     )
@@
     )
   )
+  (global_label "PB3" (shape input) (at 160.02 50.8 180) (fields_autoplaced)
+    (effects (font (size 1.27 1.27)) (justify right))
+    (property "Intersheetrefs" "${INTERSHEET_REFS}" (at 153.9395 50.8 0)
+      (effects (font (size 1.27 1.27)) (justify right) hide)
+    )
+  )
   (global_label "PB0{slash}MOSI" (shape input) (at 99.06 44.45 0) (fields_autoplaced)
     (effects (font (size 1.27 1.27)) (justify left))
@@
     )
   )
+  (symbol (lib_id "Connector:Conn_01x03_Pin") (at 155.702 75.946 0) (unit 1)
+    (in_bom yes) (on_board yes) (dnp no) (fields_autoplaced)
+    (property "Reference" "J2" (at 156.337 68.58 0)
+      (effects (font (size 1.27 1.27)))
+    )
+    (property "Value" "Conn_01x03_Pin" (at 156.337 71.12 0)
+      (effects (font (size 1.27 1.27)))
+    )
+    (property "Footprint" "Connector_PinHeader_1.27mm:PinHeader_1x03_P1.27mm_Vertical" (at 155.702 75.946 0)
+      (effects (font (size 1.27 1.27)) hide)
+    )
+    (property "Datasheet" "~" (at 155.702 75.946 0)
+      (effects (font (size 1.27 1.27)) hide)
+    )
+    (pin "2")
+    (pin "1")
+    (pin "3")
+    (instances
+      (project "NeepNeep-DAC-V2"
+        (path "/53b8c8d9-463f-4715-b30d-544c8cc3c6e0"
+          (reference "J2") (unit 1)
+        )
+      )
+    )
+  )
   (symbol (lib_id "power:GND") (at 179.07 54.61 0) (unit 1)
     (in_bom yes) (on_board yes) (dnp no)
@@
     )
     (property "Value" "GND" (at 179.197 59.0042 0)
-      (effects (font (size 1.27 1.27)))
+      (effects (font (size 1.27 1.27)) hide)
     )
     (property "Footprint" "" (at 179.07 54.61 0)
@@
     )
   )
+  (symbol (lib_id "power:+3.3V") (at 160.782 73.406 0) (unit 1)
+    (in_bom yes) (on_board yes) (dnp no)
+    (property "Reference" "#PWR08" (at 160.782 77.216 0)
+      (effects (font (size 1.27 1.27)) hide)
+    )
+    (property "Value" "+3.3V" (at 161.163 69.0118 0)
+      (effects (font (size 1.27 1.27)))
+    )
+    (property "Footprint" "" (at 160.782 73.406 0)
+      (effects (font (size 1.27 1.27)) hide)
+    )
+    (property "Datasheet" "" (at 160.782 73.406 0)
+      (effects (font (size 1.27 1.27)) hide)
+    )
+    (pin "1")
+    (instances
+      (project "NeepNeep-DAC-V2"
+        (path "/53b8c8d9-463f-4715-b30d-544c8cc3c6e0"
+          (reference "#PWR08") (unit 1)
+        )
+      )
+    )
+  )
   (symbol (lib_id "power:GND") (at 84.328 111.506 0) (unit 1)
     (in_bom yes) (on_board yes) (dnp no)
@@
         (path "/53b8c8d9-463f-4715-b30d-544c8cc3c6e0"
           (reference "R4") (unit 1)
-        )
-      )
-    )
-  )
-  (symbol (lib_id "power:GND") (at 31.75 145.288 0) (unit 1)
-    (in_bom yes) (on_board yes) (dnp no)
-    (property "Reference" "#PWR06" (at 31.75 151.638 0)
-      (effects (font (size 1.27 1.27)) hide)
-    )
-    (property "Value" "GND" (at 31.877 149.6822 0)
-      (effects (font (size 1.27 1.27)) hide)
-    )
-    (property "Footprint" "" (at 31.75 145.288 0)
-      (effects (font (size 1.27 1.27)) hide)
-    )
-    (property "Datasheet" "" (at 31.75 145.288 0)
-      (effects (font (size 1.27 1.27)) hide)
-    )
-    (pin "1")
-    (instances
-      (project "NeepNeep-DAC-V2"
-        (path "/53b8c8d9-463f-4715-b30d-544c8cc3c6e0"
-          (reference "#PWR06") (unit 1)
         )
       )
@@
     )
   )
-  (symbol (lib_id "Jumper:Jumper_2_Open") (at 31.75 140.208 90) (unit 1)
-    (in_bom yes) (on_board yes) (dnp no) (fields_autoplaced)
-    (property "Reference" "JP1" (at 33.528 138.938 90)
-      (effects (font (size 1.27 1.27)) (justify right))
-    )
-    (property "Value" "Jumper_2_Open" (at 33.528 141.478 90)
-      (effects (font (size 1.27 1.27)) (justify right))
-    )
-    (property "Footprint" "Connector_PinSocket_1.27mm:PinSocket_1x02_P1.27mm_Vertical" (at 31.75 140.208 0)
-      (effects (font (size 1.27 1.27)) hide)
-    )
-    (property "Datasheet" "~" (at 31.75 140.208 0)
-      (effects (font (size 1.27 1.27)) hide)
-    )
-    (pin "2")
-    (pin "1")
-    (instances
-      (project "NeepNeep-DAC-V2"
-        (path "/53b8c8d9-463f-4715-b30d-544c8cc3c6e0"
-          (reference "JP1") (unit 1)
-        )
-      )
-    )
-  )
   (symbol (lib_id "power:GND") (at 105.41 90.17 0) (unit 1)
     (in_bom yes) (on_board yes) (dnp no)
@@
         )
       )
+    )
+  )
+  (symbol (lib_id "power:GND") (at 160.782 78.486 0) (unit 1)
+    (in_bom yes) (on_board yes) (dnp no)
+    (property "Reference" "#PWR09" (at 160.782 84.836 0)
+      (effects (font (size 1.27 1.27)) hide)
+    )
+    (property "Value" "GND" (at 160.909 82.8802 0)
+      (effects (font (size 1.27 1.27)) hide)
+    )
+    (property "Footprint" "" (at 160.782 78.486 0)
+      (effects (font (size 1.27 1.27)) hide)
+    )
+    (property "Datasheet" "" (at 160.782 78.486 0)
+      (effects (font (size 1.27 1.27)) hide)
+    )
+    (pin "1")
+    (instances
+      (project "NeepNeep-DAC-V2"
+        (path "/53b8c8d9-463f-4715-b30d-544c8cc3c6e0"
+          (reference "#PWR09") (unit 1)
+        )
+      )

Commit message: Commit: M	README.md A	V2/NeepNeep-DAC-V2-backups/NeepNeep-DAC-V2-2026-02-12_124743.zip A	V2/NeepNeep-DAC-V2-backups/NeepNeep-DAC-V2-2026-02-12_132550.zip A	V2/NeepNeep-DAC-V2-backups/NeepNeep-DAC-V2-2026-02-12_133556.zip A	V2/NeepNeep-DAC-V2-backups/NeepNeep-DAC-V2-2026-02-12_142149.zip A	V2/NeepNeep-DAC-V2-backups/NeepNeep-DAC-V2-2026-02-12_143905.zip A	V2/NeepNeep-DAC-V2-backups/NeepNeep-DAC-V2-2026-02-12_170144.zip M	V2/NeepNeep-DAC-V2.kicad_pcb M	V2/NeepNeep-DAC-V2.kicad_prl M	V2/NeepNeep-DAC-V2.kicad_pro M	V2/NeepNeep-DAC-V2.kicad_sch A	V2/bom/NeepNeep-DAC-V2-ibom.html M	V2/fp-info-cache A	V2/ibom.config.ini A	V2/jlcpcb/gerber/NeepNeep-DAC-V2-CuBottom.gbr A	V2/jlcpcb/gerber/NeepNeep-DAC-V2-CuTop.gbr A	V2/jlcpcb/gerber/NeepNeep-DAC-V2-EdgeCuts.gbr A	V2/jlcpcb/gerber/NeepNeep-DAC-V2-MaskBottom.gbr A	V2/jlcpcb/gerber/NeepNeep-DAC-V2-MaskTop.gbr A	V2/jlcpcb/gerber/NeepNeep-DAC-V2-NPTH-drl_map.pdf A	V2/jlcpcb/gerber/NeepNeep-DAC-V2-NPTH.drl A	V2/jlcpcb/gerber/NeepNeep-DAC-V2-PTH-drl_map.pdf A	V2/jlcpcb/gerber/NeepNeep-DAC-V2-PTH.drl A	V2/jlcpcb/gerber/NeepNeep-DAC-V2-PasteBottom.gbr A	V2/jlcpcb/gerber/NeepNeep-DAC-V2-PasteTop.gbr A	V2/jlcpcb/gerber/NeepNeep-DAC-V2-SilkBottom.gbr A	V2/jlcpcb/gerber/NeepNeep-DAC-V2-SilkTop.gbr A	V2/jlcpcb/gerber/NeepNeep-DAC-V2-VScore.gbr A	V2/jlcpcb/production_files/BOM-NeepNeep-DAC-V2.csv A	V2/jlcpcb/production_files/CPL-NeepNeep-DAC-V2.csv A	V2/jlcpcb/production_files/GERBER-NeepNeep-DAC-V2.zip A	V2/jlcpcb/project.db
Parts:
- J1: footprint Global Kicad FootprintLibrary:PRG-Header_1x06_P1.27mm -> Niffum-Connector:SPI-Header_1x06_P1.27mm
- J2: footprint Connector_PinHeader_1.27mm:PinHeader_1x03_P1.27mm_Vertical -> Niffum-Connector:UPDI PinHeader_1x03_P1.27mm_Vertical
- renumbered U3 to U1
Connections:
- net +3V3: now also J1.1 (Pin_1), J2.3 (Pin_3); no longer J1.2 (Pin_2), J2.1 (Pin_1)
- net GND: now also J1.2 (Pin_2), J2.1 (Pin_1); no longer J1.6 (Pin_6), J2.3 (Pin_3)
- net PB0/MOSI: now also J1.5 (Pin_5); no longer J1.4 (Pin_4)
- net PB1/MISO: now also J1.4 (Pin_4); no longer J1.1 (Pin_1)
- net PB2/SCK: now also J1.6 (Pin_6); no longer J1.3 (Pin_3)
- net PB3: now also J1.3 (Pin_3); no longer J1.5 (Pin_5)
Changed lines of the file:
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@@
-    (stroke (width 0) (type default))
-  )
-  (wire (pts (xy 172.72 45.72) (xy 179.07 45.72))
     (stroke (width 0) (type default))
   )
@@
     (stroke (width 0) (type default))
   )
+  (wire (pts (xy 153.924 45.72) (xy 160.02 45.72))
+    (stroke (width 0) (type default))
+  )
   (wire (pts (xy 71.882 103.886) (xy 71.882 101.346))
     (stroke (width 0) (type default))
@@
     (stroke (width 0) (type default))
   )
-  (wire (pts (xy 172.72 50.8) (xy 179.07 50.8))
-    (stroke (width 0) (type default))
-  )
   (wire (pts (xy 203.962 34.036) (xy 218.694 34.036))
     (stroke (width 0) (type default))
@@
     (stroke (width 0) (type default))
   )
+  (wire (pts (xy 153.924 43.434) (xy 153.924 45.72))
+    (stroke (width 0) (type default))
+  )
   (wire (pts (xy 203.962 44.45) (xy 218.694 44.45))
     (stroke (width 0) (type default))
@@
     (stroke (width 0) (type default))
   )
-  (wire (pts (xy 179.07 50.8) (xy 179.07 54.61))
-    (stroke (width 0) (type default))
-  )
   (wire (pts (xy 218.694 26.416) (xy 218.694 34.036))
     (stroke (width 0) (type default))
@@
   )
   (wire (pts (xy 218.694 39.624) (xy 218.694 44.45))
-    (stroke (width 0) (type default))
-  )
-  (wire (pts (xy 179.07 45.72) (xy 179.07 40.64))
     (stroke (width 0) (type default))
   )
@@
     )
   )
-  (global_label "PB0{slash}MOSI" (shape input) (at 172.72 48.26 0) (fields_autoplaced)
-    (effects (font (size 1.27 1.27)) (justify left))
-    (property "Intersheetrefs" "${INTERSHEET_REFS}" (at 184.7272 48.26 0)
-      (effects (font (size 1.27 1.27)) (justify left) hide)
+  (global_label "PB0{slash}MOSI" (shape input) (at 160.02 50.8 180) (fields_autoplaced)
+    (effects (font (size 1.27 1.27)) (justify right))
+    (property "Intersheetrefs" "${INTERSHEET_REFS}" (at 148.0128 50.8 0)
+      (effects (font (size 1.27 1.27)) (justify right) hide)
     )
   )
@@
     )
   )
-  (global_label "PB1{slash}MISO" (shape input) (at 160.02 45.72 180) (fields_autoplaced)
+  (global_label "PB1{slash}MISO" (shape input) (at 172.72 48.26 0) (fields_autoplaced)
+    (effects (font (size 1.27 1.27)) (justify left))
+    (property "Intersheetrefs" "${INTERSHEET_REFS}" (at 184.7272 48.26 0)
+      (effects (font (size 1.27 1.27)) (justify left) hide)
+    )
+  )
+  (global_label "PB3" (shape input) (at 160.02 48.26 180) (fields_autoplaced)
     (effects (font (size 1.27 1.27)) (justify right))
-    (property "Intersheetrefs" "${INTERSHEET_REFS}" (at 148.0128 45.72 0)
-      (effects (font (size 1.27 1.27)) (justify right) hide)
-    )
-  )
-  (global_label "PB3" (shape input) (at 160.02 50.8 180) (fields_autoplaced)
-    (effects (font (size 1.27 1.27)) (justify right))
-    (property "Intersheetrefs" "${INTERSHEET_REFS}" (at 153.9395 50.8 0)
+    (property "Intersheetrefs" "${INTERSHEET_REFS}" (at 153.9395 48.26 0)
       (effects (font (size 1.27 1.27)) (justify right) hide)
     )
@@
     )
   )
-  (global_label "PB2{slash}SCK" (shape input) (at 160.02 48.26 180) (fields_autoplaced)
-    (effects (font (size 1.27 1.27)) (justify right))
-    (property "Intersheetrefs" "${INTERSHEET_REFS}" (at 148.8595 48.26 0)
-      (effects (font (size 1.27 1.27)) (justify right) hide)
+  (global_label "PB2{slash}SCK" (shape input) (at 172.72 50.8 0) (fields_autoplaced)
+    (effects (font (size 1.27 1.27)) (justify left))
+    (property "Intersheetrefs" "${INTERSHEET_REFS}" (at 183.8805 50.8 0)
+      (effects (font (size 1.27 1.27)) (justify left) hide)
     )
   )
@@
     )
   )
-  (symbol (lib_id "Connector:Conn_01x03_Pin") (at 155.702 75.946 0) (unit 1)
-    (in_bom yes) (on_board yes) (dnp no) (fields_autoplaced)
-    (property "Reference" "J2" (at 156.337 68.58 0)
+  (symbol (lib_id "Connector:Conn_01x03_Pin") (at 155.702 75.946 0) (mirror x) (unit 1)
+    (in_bom yes) (on_board yes) (dnp no)
+    (property "Reference" "J2" (at 156.337 83.312 0)
       (effects (font (size 1.27 1.27)))
     )
-    (property "Value" "Conn_01x03_Pin" (at 156.337 71.12 0)
+    (property "Value" "Conn_01x03_Pin" (at 156.337 80.772 0)
       (effects (font (size 1.27 1.27)))
     )
-    (property "Footprint" "Connector_PinHeader_1.27mm:PinHeader_1x03_P1.27mm_Vertical" (at 155.702 75.946 0)
+    (property "Footprint" "Niffum-Connector:UPDI PinHeader_1x03_P1.27mm_Vertical" (at 155.702 75.946 0)
       (effects (font (size 1.27 1.27)) hide)
     )
@@
     )
   )
-  (symbol (lib_id "power:GND") (at 179.07 54.61 0) (unit 1)
-    (in_bom yes) (on_board yes) (dnp no)
-    (property "Reference" "#PWR0113" (at 179.07 60.96 0)
-      (effects (font (size 1.27 1.27)) hide)
-    )
-    (property "Value" "GND" (at 179.197 59.0042 0)
-      (effects (font (size 1.27 1.27)) hide)
-    )
-    (property "Footprint" "" (at 179.07 54.61 0)
-      (effects (font (size 1.27 1.27)) hide)
-    )
-    (property "Datasheet" "" (at 179.07 54.61 0)
+  (symbol (lib_id "power:GND") (at 172.72 45.72 90) (unit 1)
+    (in_bom yes) (on_board yes) (dnp no)
+    (property "Reference" "#PWR0113" (at 179.07 45.72 0)
+      (effects (font (size 1.27 1.27)) hide)
+    )
+    (property "Value" "GND" (at 177.1142 45.593 0)
+      (effects (font (size 1.27 1.27)) hide)
+    )
+    (property "Footprint" "" (at 172.72 45.72 0)
+      (effects (font (size 1.27 1.27)) hide)
+    )
+    (property "Datasheet" "" (at 172.72 45.72 0)
       (effects (font (size 1.27 1.27)) hide)
     )
@@
   (symbol (lib_id "MCU_Microchip_ATtiny:ATtiny85-20S") (at 83.82 52.07 0) (unit 1)
     (in_bom yes) (on_board yes) (dnp no)
-    (property "Reference" "U3" (at 89.662 31.242 0)
+    (property "Reference" "U1" (at 89.662 31.242 0)
       (effects (font (size 1.27 1.27)) (justify left))
     )
@@
       (project "NeepNeep-DAC-V2"
         (path "/53b8c8d9-463f-4715-b30d-544c8cc3c6e0"
-          (reference "U3") (unit 1)
+          (reference "U1") (unit 1)
         )
       )
@@
       (effects (font (size 1.27 1.27)))
     )
-    (property "Footprint" "Global Kicad FootprintLibrary:PRG-Header_1x06_P1.27mm" (at 165.1 48.26 0)
+    (property "Footprint" "Niffum-Connector:SPI-Header_1x06_P1.27mm" (at 165.1 48.26 0)
       (effects (font (size 1.27 1.27)) hide)
     )
@@
     )
   )
-  (symbol (lib_id "power:+3.3V") (at 179.07 40.64 0) (unit 1)
-    (in_bom yes) (on_board yes) (dnp no)
-    (property "Reference" "#PWR0110" (at 179.07 44.45 0)
-      (effects (font (size 1.27 1.27)) hide)
-    )
-    (property "Value" "+3.3V" (at 179.451 36.2458 0)
+  (symbol (lib_id "power:+3.3V") (at 153.924 43.434 0) (unit 1)
+    (in_bom yes) (on_board yes) (dnp no)
+    (property "Reference" "#PWR0110" (at 153.924 47.244 0)
+      (effects (font (size 1.27 1.27)) hide)
+    )
+    (property "Value" "+3.3V" (at 154.305 39.0398 0)
       (effects (font (size 1.27 1.27)))
     )
-    (property "Footprint" "" (at 179.07 40.64 0)
-      (effects (font (size 1.27 1.27)) hide)
-    )
-    (property "Datasheet" "" (at 179.07 40.64 0)
-      (effects (font (size 1.27 1.27)) hide)
-    )
+    (property "Footprint" "" (at 153.924 43.434 0)
+      (effects (font (size 1.27 1.27)) hide)
+    )
+    (property "Datasheet" "" (at 153.924 43.434 0)
+      (effects (font (size 1.27 1.27)) hide)
+    )

Commit message: Commit: D	V2/NeepNeep-DAC-V2-backups/NeepNeep-DAC-V2-2026-02-12_132550.zip A	V2/NeepNeep-DAC-V2-backups/NeepNeep-DAC-V2-2026-02-13_132614.zip A	V2/NeepNeep-DAC-V2-backups/NeepNeep-DAC-V2-2026-02-13_133905.zip A	V2/NeepNeep-DAC-V2-backups/NeepNeep-DAC-V2-2026-02-13_135245.zip A	V2/NeepNeep-DAC-V2-backups/NeepNeep-DAC-V2-2026-02-13_140056.zip A	V2/NeepNeep-DAC-V2-backups/NeepNeep-DAC-V2-2026-02-13_141120.zip M	V2/NeepNeep-DAC-V2.kicad_pcb M	V2/NeepNeep-DAC-V2.kicad_sch
Parts:
- removed U1: ATtiny85-20SU, Package_SO:SOIC-8W_5.3x5.3mm_P1.27mm, symbol MCU_Microchip_ATtiny:ATtiny85-20S
- added U1: ATtiny412-SS, Package_SO:SOIC-8_3.9x4.9mm_P1.27mm, symbol MCU_Microchip_ATtiny:ATtiny412-SS
Connections:
- net +3V3: now also U1.1 (VCC)
- net GND: now also U1.8 (GND)
- net PB0/MOSI renamed FLASH_DI
- net FLASH_DI: now also U1.4 (PA1)
- net PB1/MISO renamed FLASH_DO
- net FLASH_DO: now also U1.5 (PA2)
- net PB2/SCK renamed FLASH_CLK
- net FLASH_CLK: now also U1.7 (PA3)
- net PB3 renamed FLASH_CS
- net FLASH_CS: now also U1.2 (PA6)
- net PB4 renamed SPEAKER
- net SPEAKER: now also U1.3 (PA7)
- net PB5/RESET renamed RESET
- net RESET: now also U1.6 (~{RESET}/PA0)
Other:
- note added: "ATtiny412 SPI Pins PA1: SPI MOSI -> DI PA2: SPI MISO -> DO PA3: SPI SCK"
- note removed: "Idealy i woudl like to use an ATTINY85-20SU that has 8k of flash, SOIC package but they are pretty pricy right now. The ATTINY45-20SU/ATTINY45-20SUR is probably an ok intermediate as its the same as the 85 except it has 4k of flash. I belive it has two timers aswell?? JLCPCB seems to have toe 20SUR version at $1.9 and the 20SU at $3.45, not sure why??? The ATTINY13A-SSUR is pretty cheap but fuck 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"
- note removed: "Loading data.. Uno ICSP → ATtiny Pins VCC → Pin 8 GND → Pin 4 MOSI → Pin 5 (PB0) MISO → Pin 6 (PB1) SCK → Pin 7 (PB2) RESET → Pin 1 (PB5) Program the AtTiny85 with special code so that i can load the data onto the W25. / Simple SPI flash programmer (adapt from GitHub examples) void setup() { /* Serial USB init */ } void loop() { if(Serial.available()) { uint32_t addr = /* parse addr */; spi_cs_lo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"
